File: schematic/F#32.kicad_sch (KiCad schematic)
At the start: 3 parts

Commit message: continued schematic
Parts:
- added M?: Stepper, symbol Motor:Stepper_Motor_bipolar
- added R? (x4): R, symbol Device:R
- added SW?: SW_DIP_x04, symbol Switch:SW_DIP_x04
- added SW?: MenuBtn, symbol Switch:SW_Push
- added SW?: BackBtn, symbol Switch:SW_Push
- added U?: MAX232, symbol Interface_UART:MAX232
- added U? (x3): TLC3702, symbol Amplifier_Operational:TLC272
- added U?: MP7524, symbol Flo:MP7524
- added U?: SSD1306, symbol Flo:SSD1306
Connections:
- net +5V: now also R?.2, R?.2, U?.14 (Vcc), U?.15 (Vref), U?.2 (VCC), U?.8 (V+)
- net GND: now also R?.2, R?.2, SW?.1, SW?.1, SW?.5, SW?.6, SW?.7, SW?.8, U?.1 (GND), U?.3 (GND), U?.4 (V-)
- net Rx: now reaches U?.14 (PD0)
- net Tx: now reaches U?.15 (PD1)
- net PhaseA: now reaches U?.16 (PD2)
- net PhaseA: now also U?.7
- net PhaseB: now reaches U?.17 (PD3)
- net PhaseB: now also U?.1
- net Row0: now reaches U?.18 (PD4)
- net Row0: now also M?.9 (r0)
- net Row1: now reaches U?.19 (PD5)
- net Row1: now also M?.10 (r1)
- net Row2: now reaches U?.20 (PD6)
- net Row2: now also M?.11 (r2)
- net Row3: now reaches U?.21 (PD7)
- net Row3: now also M?.12 (r3)
- net SCL: now reaches U?.22 (PC0)
- net SCL: now also U?.3 (SCL)
- net SDA: now reaches U?.23 (PC1)
- net SDA: now also U?.4 (SDA)
- net OctaveSetting0: now reaches U?.24 (PC2)
- net OctaveSetting0: now also SW?.1
- net OctaveSetting1: now reaches U?.25 (PC3)
- net OctaveSetting1: now also SW?.2
- net Vivrato: now reaches U?.26 (PC4)
- net Vivrato: now also SW?.3
- net Tremolo: now reaches U?.27 (PC5)
- net Tremolo: now also SW?.4
- net MenuBtn: now reaches U?.28 (PC6)
- net MenuBtn: now also SW?.2
- net BackBtn: now reaches U?.29 (PC7)
- net BackBtn: now also SW?.2
- net at U?.33 (PA7): now also U?.11 (DB0); no longer M?.12 (r3)
- net at U?.34 (PA6): now also U?.10 (DB1); no longer M?.11 (r2)
- net at U?.35 (PA5): now also U?.9 (DB2); no longer M?.10 (r1)
- net at U?.36 (PA4): now also U?.8 (DB3); no longer M?.9 (r0)
- net at U?.37 (PA3): now also U?.7 (DB4)
- net at U?.38 (PA2): now also U?.6 (DB5)
- net at U?.39 (PA1): now also U?.5 (DB6)
- net at U?.40 (PA0): now also U?.4 (DB7)
- net MOSI: now reaches M?.6 (c5), U?.6 (PB5)
- net MISO: now reaches M?.7 (c6), U?.7 (PB6)
- net CLK: now reaches M?.8 (c7), U?.8 (PB7)
- net RESET: now reaches R?.2, U?.9 (~{RESET})
- new net: M?.4, R?.1, R?.1, U?.2 (-)
- new net: M?.1, R?.1, R?.1, U?.6 (-)
- new net: M?.2 (-), U?.5 (+)
- new net: M?.3, U?.3 (+)
- no-connect marks 0 -> 3
Other:
- moved on the sheet: R?, U?
