File: schematic/FSharp32.kicad_pcb (KiCad board)
At the start: 2 copper layers, 301 x 40.6 mm, 78 parts, among them J1 SerialPort, J2 PICkit2, J3 AudioJack2_Ground, J4 POWER, J5 MatrixCols, J6 MatrixRows, M1 Stepper, SW2 MENU, SW3 BACK, U1 TLC3702, U2 MAX232, U3 MCP6002-xSN, U4 ATmega32-16P, U5 SSD1306, U6 LM4861, Y1 16M

Commit message: pcb progress
Parts:
- added ?: SolderWire-0.1sqmm_1x01_D0.4mm_OD1mm, Connector_Wire:SolderWire-0.1sqmm_1x01_D0.4mm_OD1mm, F.Cu at (268.0, -180.3)
- added ?: SolderWire-0.1sqmm_1x01_D0.4mm_OD1mm, Connector_Wire:SolderWire-0.1sqmm_1x01_D0.4mm_OD1mm, F.Cu at (268.0, -214.6)
- added ?: SolderWire-0.1sqmm_1x01_D0.4mm_OD1mm, Connector_Wire:SolderWire-0.1sqmm_1x01_D0.4mm_OD1mm, F.Cu at (-26.7, -214.6)
- added ?: SolderWire-0.1sqmm_1x01_D0.4mm_OD1mm, Connector_Wire:SolderWire-0.1sqmm_1x01_D0.4mm_OD1mm, F.Cu at (-26.7, -180.3)
- added ?: , , F.Cu at (-26.7, -214.6)
- added ?: , , F.Cu at (-26.7, -180.3)
- DISTORTION1: footprint Connector_PinHeader_2.54mm:PinHeader_1x03_P2.54mm_Vertical -> Connector_PinSocket_2.54mm:PinSocket_1x02_P2.54mm_Vertical
- J1: renamed from J2; footprint Connector_PinHeader_2.54mm:PinHeader_1x06_P2.54mm_Vertical -> Connector_PinSocket_2.54mm:PinSocket_1x06_P2.54mm_Horizontal
- J3: renamed from J5; footprint Connector_PinHeader_2.54mm:PinHeader_1x08_P2.54mm_Vertical -> Connector_PinSocket_2.54mm:PinSocket_1x08_P2.54mm_Vertical
- J4: renamed from J6; footprint Connector_PinHeader_2.54mm:PinHeader_1x04_P2.54mm_Vertical -> Connector_PinSocket_2.54mm:PinSocket_1x04_P2.54mm_Vertical
- L2, L3, L4, L5: footprint Inductor_THT:L_Axial_L5.3mm_D2.2mm_P7.62mm_Horizontal_Vishay_IM-1 -> Inductor_THT:L_Axial_L6.6mm_D2.7mm_P10.16mm_Horizontal_Vishay_IM-2
- SW2, SW3: footprint Connector_PinHeader_2.54mm:PinHeader_1x02_P2.54mm_Vertical -> Connector_PinSocket_2.54mm:PinSocket_1x02_P2.54mm_Vertical
- U3: footprint Connector_PinHeader_2.54mm:PinHeader_1x03_P2.54mm_Vertical -> Package_SO:SOIC-8_3.9x4.9mm_P1.27mm
- U5: footprint Connector_PinHeader_2.54mm:PinHeader_1x04_P2.54mm_Vertical -> Connector_PinSocket_2.54mm:PinSocket_1x04_P2.54mm_Vertical
- VOLUME: renamed from VOLUME1; footprint Connector_PinHeader_2.54mm:PinHeader_1x03_P2.54mm_Vertical -> Connector_PinSocket_2.54mm:PinSocket_1x03_P2.54mm_Vertical
- moved R20 421.3 mm to (224.8, -206.6), turned to 90 degrees
- moved C21 413.4 mm to (228.6, -213.3)
- moved C19 413.1 mm to (222.2, -206.6), turned to -90 degrees
- moved LS1 389.7 mm to (261.6, -231.0)
- moved J5 388.3 mm to (256.7, -215.8)
- moved U6 370.3 mm to (229.9, -207.6)
- moved VOLUME 363.2 mm to (232.4, -201.8), turned to -90 degrees
- moved SW6 307.8 mm to (289.6, -184.8), turned to 180 degrees
- moved C18 259.1 mm to (163.8, 248.9), turned to 180 degrees
- moved C17 259.0 mm to (163.8, 245.1), turned to 180 degrees
- moved C16 258.9 mm to (163.8, 241.3), turned to 180 degrees
- moved C15 258.8 mm to (163.8, 237.5), turned to 180 degrees
- moved C14 258.7 mm to (163.8, 233.7), turned to 180 degrees
- moved R10 257.4 mm to (132.1, 141.0)
- moved L3 255.8 mm to (166.4, 237.5)
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- renumbered C2 to C1, C8 to C10, C9 to C11, C10 to C12, C11 to C13, C12 to C14, C13 to C15, C14 to C16, C15 to C17, C16 to C18, C17 to C19, C1 to C2, C18 to C20, C19 to C21, C20 to C4, C21 to C5, C4 to C6, C5 to C7, C6 to C8, C7 to C9, J1 to J2, J3 to J5, J4 to J6, R11 to R10, R12 to R11, R13 to R12, R14 to R13, R15 to R14, R16 to R15, R17 to R16, R18 to R17, R19 to R18, R20 to R19, R21 to R20, R22 to R21, R23 to R22, R24 to R23, R25 to R24, R26 to R25, R27 to R26, R28 to R27, R29 to R28, R8 to R7, R9 to R8, R10 to R9
Connections:
- C13 pad 1: Net-(C11-Pad1) -> Net-(C13-Pad1)
- C19 pad 1: Net-(U3B--) -> Net-(C19-Pad1)
- C19 pad 2: Net-(C17-Pad2) -> Net-(U3B--)
- J5 pad R: (no net) -> Net-(SW6B-C)
- R20 pad 2: Net-(C17-Pad2) -> Net-(C19-Pad1)
- VOLUME pad 1: Net-(U6--) -> Net-(SW6A-B)
- VOLUME pad 3: Net-(SW6A-B) -> Net-(U6--)
Routing:
- net Net-(C17-Pad1): track 0.00 -> 14.4 mm
- net Net-(C16-Pad1): track 0.00 -> 14.4 mm
- net Net-(C15-Pad1): track 0.00 -> 14.4 mm
- net Net-(U3B-+): track 0.00 -> 14.4 mm
- net Net-(R22-Pad2): track 0.00 -> 14.3 mm
- net Net-(R17-Pad2): track 0.00 -> 14.3 mm
- net Net-(R15-Pad2): track 0.00 -> 14.3 mm
- net Net-(R11-Pad2): track 0.00 -> 14.3 mm
- net Net-(R19-Pad2): track 0.00 -> 14.3 mm
- net Net-(C14-Pad1): track 0.00 -> 14.3 mm
- net Net-(R26-Pad2): track 0.00 -> 11.7 mm
- net Net-(R24-Pad2): track 0.00 -> 11.7 mm
- net Net-(U2-C2-): track 0.00 -> 9.43 mm
- net Net-(U2-C2+): track 0.00 -> 9.42 mm
- net +5V: track 0.00 -> 5.08 mm
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Other:
- board size 301 x 40.6 mm -> 335.9 x 40.6 mm

Commit message: continued pcb
Parts:
- removed DISTORTION1: 100k, Connector_PinSocket_2.54mm:PinSocket_1x02_P2.54mm_Vertical
- removed LS1: Speaker, TerminalBlock:TerminalBlock_bornier-2_P5.08mm
- removed SW1: ~, Connector_PinSocket_2.54mm:PinSocket_1x03_P2.54mm_Vertical
- removed SW2: MENU, Connector_PinSocket_2.54mm:PinSocket_1x02_P2.54mm_Vertical
- removed SW3: BACK, Connector_PinSocket_2.54mm:PinSocket_1x02_P2.54mm_Vertical
- removed SW4, SW5: ~, Connector_PinSocket_2.54mm:PinSocket_1x02_P2.54mm_Vertical
- removed SW6: ~, Connector_PinSocket_2.54mm:PinSocket_2x03_P2.54mm_Vertical
- removed VOLUME: 1k, Connector_PinSocket_2.54mm:PinSocket_1x03_P2.54mm_Vertical
- added ?: , , F.Cu at (226.7, 52.1)
- added ?: , , F.Cu at (199.4, 29.2)
- added ?: , , F.Cu at (196.2, 52.1)
- added ?: , , F.Cu at (226.7, 17.8)
- added ?: , , F.Cu at (276.9, 76.8)
- added ?: , , F.Cu at (271.8, 70.5)
- added ?: , , F.Cu at (199.4, 40.6)
- added ?: , , F.Cu at (199.4, 39.4)
- added ?: , , F.Cu at (196.2, 17.8)
- added ?: , , F.Cu at (265.4, 70.5)
- added ?: , , F.Cu at (276.9, 74.3)
- added ?: , , F.Cu at (199.4, 30.5)
- added REF**: SolderWirePad_1x01_SMD_1x2mm, Connector_Wire:SolderWirePad_1x01_SMD_1x2mm, F.Cu at (76.8, 95.9)
- added REF**: SolderWirePad_1x01_SMD_1x2mm, Connector_Wire:SolderWirePad_1x01_SMD_1x2mm, F.Cu at (269.4, 87.0)
- added REF**: SolderWirePad_1x01_SMD_1x2mm, Connector_Wire:SolderWirePad_1x01_SMD_1x2mm, F.Cu at (142.2, 36.2)
- added REF**: SolderWirePad_1x01_SMD_1x2mm, Connector_Wire:SolderWirePad_1x01_SMD_1x2mm, F.Cu at (68.6, 38.7)
- added REF**: SolderWirePad_1x01_SMD_1x2mm, Connector_Wire:SolderWirePad_1x01_SMD_1x2mm, F.Cu at (79.4, 38.7)
- added REF**: SolderWirePad_1x01_SMD_1x2mm, Connector_Wire:SolderWirePad_1x01_SMD_1x2mm, F.Cu at (163.2, 36.2)
- added REF**: SolderWirePad_1x01_SMD_1x2mm, Connector_Wire:SolderWirePad_1x01_SMD_1x2mm, F.Cu at (288.3, 88.3)
- C19, F1, R20, U6: moved to B.Cu
- moved C10 385.3 mm to (20.5, 67.9)
- moved C12 368.2 mm to (58.5, 113.7)
- moved C11 366.2 mm to (59.7, 137.1), turned to 90 degrees
- moved C5 362.2 mm to (65.4, 114.3), turned to 90 degrees
- moved J3 359.7 mm to (38.1, 135.9), turned to 90 degrees
- moved Y1 358.5 mm to (69.8, 136.5), turned to 180 degrees
- moved C4 358.0 mm to (69.2, 114.3), turned to 90 degrees
- moved C8 351.0 mm to (74.9, 137.2), turned to 90 degrees
- moved ? 327.2 mm to (64.1, 99.7)
- moved J4 321.2 mm to (81.3, 135.9), turned to 90 degrees
- moved U6 285.2 mm to (269.2, 74.9)
- moved ? 284.2 mm to (21.6, 99.7)
- moved C19 283.3 mm to (261.6, 74.0), turned to 90 degrees
- moved R20 283.3 mm to (264.2, 73.9), turned to -90 degrees
- moved C21 282.7 mm to (268.0, 66.7), turned to 180 degrees
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Connections:
- M1 pad 1: Net-(U1B--) -> Net-(M1-Pad1)
- R2 pad 2: Net-(M1--) -> Net-(M1-Pad1)
- R3 pad 1: Net-(U1B--) -> Net-(M1--)
- R4 pad 1: Net-(U1B--) -> Net-(M1--)
- U1 pad 6: Net-(U1B--) -> Net-(M1--)
Routing:
- net +5V: track 5.08 -> 44.4 mm
- net Row3: track 0.00 -> 20.1 mm
- net Net-(U2-R2IN): track 0.00 -> 15.5 mm
- net Net-(U2-T2OUT): track 0.00 -> 15.3 mm
- net Net-(SW6A-C): track 0.00 -> 13.2 mm
- net Net-(U3A--): track 0.00 -> 11.4 mm
- net Net-(U4-XTAL2): track 0.00 -> 10.9 mm
- net Net-(U4-XTAL1): track 0.00 -> 10.8 mm
- net Net-(U6-+): track 1.27 -> 9.90 mm
- net Net-(SW6A-B): track 0.00 -> 8.24 mm
- net Net-(U6--): track 2.67 -> 8.76 mm
- net Net-(SW6B-B): track 0.00 -> 5.15 mm
- net Net-(J3-Pin_3): track 0.00 -> 3.81 mm
- net Net-(J3-Pin_2): track 0.00 -> 3.81 mm
- net Net-(J3-Pin_1): track 0.00 -> 3.81 mm
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Other:
- board size 335.9 x 40.6 mm -> 301 x 83.8 mm
- board text added: "AM"
- board text added: "BACK"
- board text added: "DISTORTION"
- board text added: "FM"
- board text added: "MENU"
- board text added: "OCTAVE"
- board text added: "SCREEN"
- board text added: "VOLUME"
- board text added: "──"
- board text added: "󰋋"
- board text added: "󱄠"

Commit message: finished routing
Parts:
- added ?: , , F.Cu at (172.1, 83.2)
- added ?: , , F.Cu at (174.6, 83.2)
- added ?: , , F.Cu at (169.5, 85.1)
- added ?: , , F.Cu at (169.5, 87.6)
- added ?: , , F.Cu at (177.2, 83.2)
- added ?: , , F.Cu at (179.7, 83.2)
- J1: footprint Connector_PinSocket_2.54mm:PinSocket_1x06_P2.54mm_Horizontal -> Connector_PinHeader_2.54mm:PinHeader_1x06_P2.54mm_Vertical
- J2: footprint Connector_Dsub:DSUB-9_Male_Horizontal_P2.77x2.84mm_EdgePinOffset7.70mm_Housed_MountingHolesOffset9.12mm -> Connector_Dsub:DSUB-9_Male_Horizontal_P2.77x2.84mm_EdgePinOffset4.94mm_Housed_MountingHolesOffset7.48mm
- R12, R14, U3: moved to B.Cu
- moved C5 108.3 mm to (167.0, 76.8), turned to 180 degrees
- moved C12 107.5 mm to (159.4, 76.8)
- moved C11 107.5 mm to (160.7, 100.3)
- moved C8 107.5 mm to (175.9, 100.3)
- moved U4 107.5 mm to (139.1, 95.2)
- moved Y1 107.5 mm to (170.8, 99.7)
- moved J3 107.5 mm to (139.1, 99.1)
- moved J4 107.5 mm to (182.2, 99.1)
- moved C4 107.1 mm to (169.5, 76.8), turned to 0 degrees
- moved REF** 104.8 mm to (69.2, 82.5)
- moved J2 97.2 mm to (125.8, 70.2)
- moved C3 93.2 mm to (127.0, 78.1), turned to 90 degrees
- moved J6 93.2 mm to (188.6, 64.8), turned to 180 degrees
- moved C2 92.8 mm to (132.7, 95.2), turned to 180 degrees
- moved C7 89.7 mm to (121.3, 75.6)
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Connections:
- R1 pad 1: PhaseA -> PhaseB
- R5 pad 1: PhaseB -> PhaseA
- U1 pad 1: PhaseB -> PhaseA
- U1 pad 7: PhaseA -> PhaseB
Routing:
- net +5V: track 44.4 -> 406.5 mm, vias 0 -> 2
- net PhaseA: track 0.00 -> 181.4 mm
- net PhaseB: track 0.00 -> 176.3 mm
- net SCL: track 0.00 -> 101.4 mm
- net SDA: track 0.00 -> 95.2 mm
- net DAC7: track 0.00 -> 82.0 mm
- net DAC6: track 0.00 -> 80.7 mm
- net DAC5: track 0.00 -> 79.5 mm
- net Net-(L1-Pad1): track 0.00 -> 79.4 mm
- net DAC4: track 0.00 -> 78.2 mm
- net DAC3: track 0.00 -> 76.9 mm
- net DAC2: track 0.00 -> 75.7 mm
- net DAC1: track 0.00 -> 74.4 mm
- net DAC0: track 0.00 -> 73.1 mm
- net RESET: track 0.00 -> 66.8 mm
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Other:
- board size 301 x 83.8 mm -> 301 x 40.6 mm
- board text added: "󰁭"
- board text added: "󰮫"
- board text removed: "BACK"
- board text removed: "MENU"
- board text removed: "SCREEN"

Commit message: finished PCB
Parts:
- moved R14 7.85 mm to (255.9, 77.5)
- moved R12 7.85 mm to (259.7, 77.5)
- moved C2 1.27 mm to (132.7, 94.0)
Routing:
- net MOSI: track 70.1 -> 64.9 mm
- net GND: track 0.00 -> 3.07 mm, vias 0 -> 1
- net Net-(U3B-+): track 77.2 -> 74.2 mm
- net +5V: track 406.5 -> 408.5 mm
- net Net-(U3A-+): track 6.27 -> 7.92 mm
- added copper zone on B.Cu, net GND
- added copper zone on F.Cu, net GND
Other:
- board text added: "<"
- board text added: "Amplifier"
- board text added: "Back"
- board text added: "CPU"
- board text added: "DAC"
- board text added: "Display"
- board text added: "Encoder"
- board text added: "F#32"
- board text added: "Filter"
- board text added: "Flofrost"
- board text added: "MODULATOR"
- board text added: "Matrix Columns"
- board text added: "Matrix Rows"
- board text added: "Menu"
- board text added: "Oct0"
- board text added: "Oct1"
- board text added: "Serial"
- board text added: "Spk+"
- board text added: "Spk-"
- board text added: "Volume"

Commit message: fully finished pcb and order placed
Parts:
- removed the ? at (255.3, 65.4)
- removed the ? at (255.3, 99.7)
- J2: footprint Connector_Dsub:DSUB-9_Male_Horizontal_P2.77x2.84mm_EdgePinOffset4.94mm_Housed_MountingHolesOffset7.48mm -> Connector_Dsub:DSUB-9_Female_Horizontal_P2.77x2.84mm_EdgePinOffset7.70mm_Housed_MountingHolesOffset9.12mm
- moved ? 280.9 mm to (72.4, 269.9), turned to -90 degrees
- moved ? 278.6 mm to (106.7, 269.9), turned to -90 degrees
- moved REF** 268.3 mm to (85.1, 262.3), turned to -90 degrees
- moved J5 262.6 mm to (107.8, 258.4), turned to -90 degrees
- moved ? 251.5 mm to (95.2, 250.8), turned to -90 degrees
- moved ? 251.5 mm to (97.8, 250.8), turned to -90 degrees
- moved C9 249.9 mm to (106.7, 249.6), turned to 180 degrees
- moved ? 244.3 mm to (101.6, 245.7), turned to -90 degrees
- moved REF** 241.7 mm to (85.1, 243.4), turned to -90 degrees
- moved U6 240.7 mm to (97.2, 243.2), turned to -90 degrees
- moved C21 239.0 mm to (105.4, 241.9), turned to 90 degrees
- moved ? 235.3 mm to (101.6, 239.4), turned to -90 degrees
- moved R20 233.5 mm to (98.1, 238.1), turned to 180 degrees
- moved C19 229.9 mm to (98.1, 235.6), turned to 0 degrees
- moved C20 227.4 mm to (105.4, 233.7), turned to -90 degrees
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Routing:
- net Net-(U3A--): track 49.2 -> 45.9 mm
- net Net-(L1-Pad1): track 79.4 -> 76.6 mm
- net Net-(U2-T2OUT): track 13.4 -> 11.7 mm
- net Net-(C13-Pad2): track 11.4 -> 10.2 mm
- net +5V: track 408.5 -> 407.6 mm
- net Net-(U2-R2IN): track 13.3 -> 13.9 mm
Other:
- board size 301 x 40.6 mm -> 40.6 x 301 mm
- board text added: "JLCJLCJLCJLC"
