File: schematic/FSharp32.kicad_sch (KiCad schematic)
At the start: 78 parts, among them J1 PICkit2, J2 SerialPort, J3 MatrixCols, J4 MatrixRows, J5 AudioJack2_Ground, J6 POWER, M1 Stepper, SW2 MENU, SW3 BACK, U1 TLC3702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

Commit message: finished routing
Parts:
- J1: footprint Connector_PinSocket_2.54mm:PinSocket_1x06_P2.54mm_Horizontal -> Connector_PinHeader_2.54mm:PinHeader_1x06_P2.54mm_Vertical
- J2: footprint Connector_Dsub:DSUB-9_Male_Horizontal_P2.77x2.84mm_EdgePinOffset7.70mm_Housed_MountingHolesOffset9.12mm -> Connector_Dsub:DSUB-9_Male_Horizontal_P2.77x2.84mm_EdgePinOffset4.94mm_Housed_MountingHolesOffset7.48mm
Connections:
- net PhaseA: now also R5.1, U1.1; no longer R1.1, U1.7
- net PhaseB: now also R1.1, U1.7; no longer R5.1, U1.1
Changed lines of the file:
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@@
     )
   )
-  (global_label "PhaseA" (shape input) (at 107.95 29.21 180) (fields_autoplaced)
+  (global_label "PhaseA" (shape input) (at 106.68 58.42 180) (fields_autoplaced)
     (effects (font (size 1.27 1.27)) (justify right))
-    (property "Intersheetrefs" "${INTERSHEET_REFS}" (at 98.7636 29.1306 0)
+    (property "Intersheetrefs" "${INTERSHEET_REFS}" (at 97.4936 58.3406 0)
       (effects (font (size 1.27 1.27)) (justify right) hide)
     )
@@
     )
   )
-  (global_label "PhaseB" (shape input) (at 106.68 58.42 180) (fields_autoplaced)
+  (global_label "PhaseB" (shape input) (at 107.95 29.21 180) (fields_autoplaced)
     (effects (font (size 1.27 1.27)) (justify right))
-    (property "Intersheetrefs" "${INTERSHEET_REFS}" (at 97.3121 58.3406 0)
+    (property "Intersheetrefs" "${INTERSHEET_REFS}" (at 98.5821 29.1306 0)
       (effects (font (size 1.27 1.27)) (justify right) hide)
     )
@@
       (effects (font (size 1.27 1.27)) (justify left))
     )
-    (property "Footprint" "Connector_Dsub:DSUB-9_Male_Horizontal_P2.77x2.84mm_EdgePinOffset7.70mm_Housed_MountingHolesOffset9.12mm" (at 276.86 60.96 0)
+    (property "Footprint" "Connector_Dsub:DSUB-9_Male_Horizontal_P2.77x2.84mm_EdgePinOffset4.94mm_Housed_MountingHolesOffset7.48mm" (at 276.86 60.96 0)
       (effects (font (size 1.27 1.27)) hide)
     )
@@
       (effects (font (size 1.27 1.27)) (justify right))
     )
-    (property "Footprint" "Connector_PinSocket_2.54mm:PinSocket_1x06_P2.54mm_Horizontal" (at 182.88 44.45 0)
+    (property "Footprint" "Connector_PinHeader_2.54mm:PinHeader_1x06_P2.54mm_Vertical" (at 182.88 44.45 0)
       (effects (font (size 1.27 1.27)) hide)
     )

Commit message: fully finished pcb and order placed
Parts:
- J2: footprint Connector_Dsub:DSUB-9_Male_Horizontal_P2.77x2.84mm_EdgePinOffset4.94mm_Housed_MountingHolesOffset7.48mm -> Connector_Dsub:DSUB-9_Female_Horizontal_P2.77x2.84mm_EdgePinOffset7.70mm_Housed_MountingHolesOffset9.12mm
Changed lines of the file:
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@@
       (effects (font (size 1.27 1.27)) (justify left))
     )
-    (property "Footprint" "Connector_Dsub:DSUB-9_Male_Horizontal_P2.77x2.84mm_EdgePinOffset4.94mm_Housed_MountingHolesOffset7.48mm" (at 276.86 60.96 0)
+    (property "Footprint" "Connector_Dsub:DSUB-9_Female_Horizontal_P2.77x2.84mm_EdgePinOffset7.70mm_Housed_MountingHolesOffset9.12mm" (at 276.86 60.96 0)
       (effects (font (size 1.27 1.27)) hide)
     )

Commit message: did some vribrato
Parts:
- removed U4: ATmega32-16P, Package_DIP:DIP-40_W15.24mm, symbol MCU_Microchip_ATmega:ATmega32-16P
- added U4: ATmega1284-P, Package_DIP:DIP-40_W15.24mm, symbol MCU_Microchip_ATmega:ATmega1284-P
Connections:
- net +5V: now also U4.10 (VCC), U4.30 (AVCC), U4.32 (AREF)
- net BackBtn: now also U4.29 (PC7)
- net CLK: now also U4.8 (PB7)
- net DAC0: now also U4.40 (PA0)
- net DAC1: now also U4.39 (PA1)
- net DAC2: now also U4.38 (PA2)
- net DAC3: now also U4.37 (PA3)
- net DAC4: now also U4.36 (PA4)
- net DAC5: now also U4.35 (PA5)
- net DAC6: now also U4.34 (PA6)
- net DAC7: now also U4.33 (PA7)
- net GND: now also U4.11 (GND), U4.31 (GND)
- net MISO: now also U4.7 (PB6)
- net MOSI: now also U4.6 (PB5)
- net MenuBtn: now also U4.28 (PC6)
- net OctaveSetting0: now also U4.24 (PC2)
- net OctaveSetting1: now also U4.25 (PC3)
- net PhaseA: now also U4.16 (PD2)
- net PhaseB: now also U4.17 (PD3)
- net RESET: now also U4.9 (~{RESET})
- net Row0: now also U4.18 (PD4)
- net Row1: now also U4.19 (PD5)
- net Row2: now also U4.20 (PD6)
- net Row3: now also U4.21 (PD7)
- net Rx: now also U4.14 (PD0)
- net SCL: now also U4.22 (PC0)
- net SDA: now also U4.23 (PC1)
- net Tremolo: now also U4.27 (PC5)
- net Tx: now also U4.15 (PD1)
- net Vibrato: now also U4.26 (PC4)
- net at J3.1 (Pin_1): now also U4.1 (PB0)
- net at C11.2, Y1.2: now also U4.12 (XTAL2)
- net at C8.2, Y1.1: now also U4.13 (XTAL1)
- net at J3.2 (Pin_2): now also U4.2 (PB1)
- net at J3.3 (Pin_3): now also U4.3 (PB2)
- net at J3.4 (Pin_4): now also U4.4 (PB3)
- net at J3.5 (Pin_5): now also U4.5 (PB4)
